Commit message: 无人机没法跟踪轨迹中的姿态

File: urdf/gates.urdf (robot description, URDF)
Before this commit: robot rpg_gate_group, 6 links, 5 joints
Links:
- added link gate_6; visual mesh filename=package://acados_nmpc_controller/asset/RPGgate.dae scale=1 1 1
- added link gate_7; visual mesh filename=package://acados_nmpc_controller/asset/RPGgate.dae scale=1 1 1
- link gate_1: geometry visual mesh filename=package://acados_nmpc_controller/asset/RPGgate.dae scale=1 1 1
- link gate_2: geometry visual mesh filename=package://acados_nmpc_controller/asset/RPGgate.dae scale=1 1 1
- link gate_3: geometry visual mesh filename=package://acados_nmpc_controller/asset/RPGgate.dae scale=1 1 1
- link gate_4: geometry visual mesh filename=package://acados_nmpc_controller/asset/RPGgate.dae scale=1 1 1
- link gate_5: geometry visual mesh filename=package://acados_nmpc_controller/asset/RPGgate.dae scale=1 1 1
Joints:
- added joint joint_gate_6: type fixed, parent world, child gate_6, origin xyz=-8 -7 6.2 rpy=0 0 1.2308
- added joint joint_gate_7: type fixed, parent world, child gate_7, origin xyz=-8 -7 2.5 rpy=0 0 1.2308
- joint joint_gate_1: origin xyz=-10 10 2.5 rpy=0 0 1.5708 -> xyz=-2 8 2.5 rpy=0 0 -0.34
- joint joint_gate_2: origin xyz=-10 -10 2.5 rpy=0 0 0.519 -> xyz=9 9 2.5 rpy=0 0 -2.355
- joint joint_gate_3: origin xyz=0 -10 2.5 rpy=0 0 0 -> xyz=10 0 2.5 rpy=0 0 3.14
- joint joint_gate_4: origin xyz=10 -10 2.5 rpy=0 0 0.785 -> xyz=8 -8 2.5 rpy=0 0 2.07
- joint joint_gate_5: origin xyz=10 0 2.5 rpy=0 0 1.5708 -> xyz=0 -10 2.5 rpy=0 0 1.5708
